File: ft231x-breakout-v11-openSX70versionSEEED.brd (EAGLE design)
At the start: 31.8 x 15.2 mm, 24 parts, among them J1 XF2L-0625-1, Q1 2N7002, U1 FTS31XS-U

Commit message: New Breakout WIP
Parts:
- C3, C4: device Seeed-Capacitor-2016:C0402 -> Common-Parts-Library-Eagle:CC0603KRX7R9BB473_CAPC1608X90
- moved R5 1.97 mm to (24.1, 7.49)
- moved C5 1.80 mm to (15.8, 12.3)
- moved R6 1.80 mm to (19.2, 12.4)
- moved U1 1.66 mm to (18.2, 7.49)
- moved R4 1.28 mm to (8.89, 2.92), turned to 90 degrees
- moved D3 1.27 mm to (6.35, 14.0)
- moved D2 1.27 mm to (6.35, 1.27)
- moved R3 1.14 mm to (8.89, 12.1), turned to 90 degrees
- moved C3 0.89 mm to (8.89, 4.70), turned to 0 degrees
- moved C4 0.52 mm to (8.89, 10.2), turned to 0 degrees
- moved C1 0.36 mm to (24.4, 2.82)
- moved R2 0.25 mm to (8.89, 6.60)
- moved R1 0.18 mm to (8.76, 8.38)
Routing:
- net 3.3V: track 0.00 -> 61.3 mm, vias 0 -> 2
- net VCC: track 0.00 -> 49.8 mm, vias 0 -> 2
- net TXD: track 0.00 -> 19.6 mm
- net DTR: track 0.00 -> 14.1 mm
- net N$2: track 0.00 -> 13.5 mm
- net RXD: track 0.00 -> 12.6 mm, vias 0 -> 2
- net N$1: track 0.00 -> 12.5 mm
- net RESET: track 0.00 -> 9.02 mm
- net CTS: track 0.00 -> 8.18 mm
- net VOUT: track 0.00 -> 7.34 mm, vias 0 -> 1
- net N$3: track 0.00 -> 5.27 mm
- net N$4: track 0.00 -> 4.64 mm
- net N$5: track 0.00 -> 3.38 mm
- net N$6: track 0.00 -> 3.32 mm
- net N$10: track 0.00 -> 3.29 mm, vias 0 -> 1

Commit message: SeeedStudio manufacturable
Parts:
- moved SJ4 7.12 mm to (19.6, 2.16), turned to 0 degrees
- moved SJ1 5.68 mm to (13.8, 2.54)
- moved C2 4.04 mm to (13.8, 1.98), turned to 90 degrees
- moved R6 2.79 mm to (22.0, 12.4)
- moved Q1 1.88 mm to (25.5, 12.5), turned to 0 degrees
- moved R5 0.36 mm to (23.9, 7.75)
- moved C3 0.13 mm to (9.02, 4.70), turned to 180 degrees
- turned C4 to 180 degrees
- turned D2 to 180 degrees
- turned D3 to 180 degrees
Routing:
- net 3.3V: track 61.3 -> 0.00 mm, vias 2 -> 0
- net VCC: track 49.8 -> 0.00 mm, vias 2 -> 0
- net TXD: track 19.6 -> 0.00 mm
- net DTR: track 14.1 -> 0.00 mm
- net N$2: track 13.5 -> 0.00 mm
- net RXD: track 12.6 -> 0.00 mm, vias 2 -> 0
- net N$1: track 12.5 -> 0.00 mm
- net RESET: track 9.02 -> 0.00 mm
- net CTS: track 8.18 -> 0.00 mm
- net VOUT: track 7.34 -> 0.00 mm, vias 1 -> 0
- net N$3: track 5.27 -> 0.00 mm
- net N$4: track 4.64 -> 0.00 mm
- net N$5: track 3.38 -> 0.00 mm
- net N$6: track 3.32 -> 0.00 mm
- net N$10: track 3.29 -> 0.00 mm, vias 1 -> 0
