File: FT232/openSX70-FTDI-232RL/openSX70-FTDI-232RL-Basic-5V_V3.brd (EAGLE design)
At the start: 25.4 x 17.3 mm, 14 parts, among them J1 687106183722, U1 FT232RLSSOP

Commit message: New FTDI versions with FT232R L and Q
Parts:
- moved C1 3.87 mm to (4.76, -6.24)
- moved C5 3.00 mm to (9.35, -6.35)
- moved JP5 2.84 mm to (-4.67, -7.77)
Routing:
- net 3.3V: track 22.5 -> 18.5 mm
- net 5V: track 45.7 -> 48.9 mm
- net POWER: track 10.9 -> 11.4 mm
