File: FT232/openSX70-FTDI-232RL/openSX70-FTDI-232RL-Basic-5V.sch (EAGLE design)
At the start: 16 parts, among them J1 687106183722, U1 FT232RLSSOP

Commit message: NEW FTDI for manufacture 232RL based on Sparkfun FTDI basic
Parts:
- removed C1: 100nf, openSX70_PATHFINDER_V5.5-SEEED_20180522:CERAMIC-100NF-50V-10%-X7R(0603)
- removed JP2: LOGO-SFESK, SparkFun:LOGO-SFESK
- removed LOGO1: OSHW-LOGOS, SparkFun-Aesthetics:OSHW-LOGOS
- removed SJ2: (no value), SparkFun:SOLDERJUMPER_2WAYS
- added S1: (no value), SparkFun-Switches:SWITCH-SPDT-SMD-RIGHT-ANGLE
Connections:
- removed net 3.3V: C1.1, SJ2.3, U1.3V3OUT
- net 5V: now also S1.O; no longer SJ2.1
- net GND: no longer C1.2
- net POWER: now also S1.P; no longer SJ2.2
Other:
- note removed: "Default 5V"
Changed lines of the file:
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@@
 <?xml version="1.0" encoding="utf-8"?>
 <!DOCTYPE eagle SYSTEM "eagle.dtd">
-<eagle version="9.0.0">
+<eagle version="9.1.0">
 <drawing>
 <settings>
@@
 <part name="C2" library="openSX70_PATHFINDER_V5.5-SEEED_20180522" deviceset="CERAMIC-100NF-50V-10%-X7R(0603)" device="" value="100nf"/>
 <part name="C5" library="Seeed-Capacitor-2016" deviceset="TANTALUM-SMD-10UF-16V-10%(AVX-A)" device="" value="10uf"/>
-<part name="C1" library="openSX70_PATHFINDER_V5.5-SEEED_20180522" deviceset="CERAMIC-100NF-50V-10%-X7R(0603)" device="" value="100nf"/>
-<part name="GND1" library="SparkFun" deviceset="GND" device=""/>
 <part name="GND2" library="SparkFun" deviceset="GND" device=""/>
-<part name="P+1" library="SparkFun" deviceset="VCC" device="" value="3.3V"/>
 <part name="FRAME1" library="SparkFun-Aesthetics" deviceset="FRAME-LETTER" device=""/>
 <part name="U1" library="SparkFun" deviceset="FT232RL" device="SSOP"/>
@@
 <part name="R1" library="openSX70_PATHFINDER_V5.5-SEEED_20180522" deviceset="SMD-RES-1K-1%-1/10W(0603)" device="" value="1K"/>
 <part name="R2" library="openSX70_PATHFINDER_V5.5-SEEED_20180522" deviceset="SMD-RES-1K-1%-1/10W(0603)" device="" value="1K"/>
-<part name="SJ2" library="SparkFun" deviceset="SOLDERJUMPER_2WAY" device="S"/>
 <part name="U$1" library="SparkFun" deviceset="5V" device=""/>
 <part name="U$3" library="SparkFun" deviceset="5V" device=""/>
 <part name="U$4" library="SparkFun" deviceset="5V" device=""/>
-<part name="JP2" library="SparkFun" deviceset="LOGO-SFE" device="SK"/>
 <part name="JP3" library="SparkFun" deviceset="FIDUCIAL" device="1X2"/>
 <part name="JP5" library="SparkFun" deviceset="FIDUCIAL" device="1X2"/>
-<part name="LOGO1" library="SparkFun-Aesthetics" deviceset="OSHW-LOGO" device="S"/>
 <part name="USB1" library="Seeed-Connector -2016" deviceset="MICRO-USB-SMD-B-(10118193-0001LF)" device="" value="10118193-0001LF"/>
 <part name="GND3" library="SparkFun" deviceset="GND" device=""/>
@@
 <part name="D1" library="Seeed-LED" deviceset="SMD-LED-CLEAR-GREEN(0603)" device="" value="GREEN-0603"/>
 <part name="D2" library="Seeed-LED-2016" deviceset="SMD-LED-CLEAR-YELLOW(0603)" device="" value="YELLOW-0603"/>
+<part name="S1" library="SparkFun-Switches" library_urn="urn:adsk.eagle:library:535" deviceset="SWITCH-SPDT" device="-SMD-RIGHT-ANGLE" package3d_urn="urn:adsk.eagle:package:40179/1"/>
 </parts>
 <sheets>
 <sheet>
 <plain>
-<wire x1="185.42" y1="109.22" x2="185.42" y2="107.188" width="0.4064" layer="94"/>
-<text x="175.26" y="96.52" size="1.778" layer="95">Default 5V</text>
 <text x="175.26" y="7.62" size="2.54" layer="104">P. Dokter, T. Klopfenstein</text>
 <text x="238.76" y="7.62" size="2.54" layer="97">v24</text>
@@
 <instance part="C2" gate="G$1" x="66.04" y="109.22" rot="R270"/>
 <instance part="C5" gate="G$1" x="76.2" y="111.76" rot="R270"/>
-<instance part="C1" gate="G$1" x="86.36" y="109.22" rot="R270"/>
-<instance part="GND1" gate="1" x="86.36" y="101.6"/>
 <instance part="GND2" gate="1" x="106.68" y="86.36"/>
-<instance part="P+1" gate="1" x="86.36" y="132.08"/>
 <instance part="FRAME1" gate="G$1" x="0" y="0"/>
 <instance part="FRAME1" gate="G$2" x="147.32" y="0"/>
@@
 <instance part="R1" gate="G$1" x="154.94" y="119.38" rot="R90"/>
 <instance part="R2" gate="G$1" x="165.1" y="119.38" rot="R90"/>
-<instance part="SJ2" gate="G$1" x="185.42" y="109.22" rot="R180"/>
 <instance part="U$1" gate="G$1" x="154.94" y="127"/>
 <instance part="U$3" gate="G$1" x="93.98" y="132.08"/>
 <instance part="U$4" gate="G$1" x="165.1" y="127"/>
-<instance part="JP2" gate="G$1" x="231.14" y="17.78"/>
 <instance part="JP3" gate="G$1" x="238.76" y="27.94"/>
 <instance part="JP5" gate="G$1" x="238.76" y="33.02"/>
-<instance part="LOGO1" gate="G$1" x="134.62" y="10.16"/>
 <instance part="USB1" gate="G$1" x="27.94" y="121.92"/>
 <instance part="GND3" gate="1" x="58.42" y="106.68" rot="R90"/>
@@
 <instance part="D1" gate="G$1" x="165.1" y="106.68" rot="R270"/>
 <instance part="D2" gate="G$1" x="154.94" y="106.68" rot="R270"/>
+<instance part="S1" gate="1" x="190.5" y="109.22" rot="R180"/>
 </instances>
 <busses>
@@
 <nets>
 <net name="GND" class="1">
-<segment>
-<wire x1="86.36" y1="105.41" x2="86.36" y2="104.14" width="0.1524" layer="91"/>
-<pinref part="GND1" gate="1" pin="GND"/>
-<pinref part="C1" gate="G$1" pin="2"/>
-</segment>
 <segment>
 <wire x1="109.22" y1="101.6" x2="106.68" y2="101.6" width="0.1524" layer="91"/>
@@
 </segment>
 </net>
-<net name="3.3V" class="1">
-<segment>
-<wire x1="86.36" y1="132.08" x2="86.36" y2="116.84" width="0.1524" layer="91"/>
-<wire x1="109.22" y1="116.84" x2="86.36" y2="116.84" width="0.1524" layer="91"/>
-<wire x1="86.36" y1="116.84" x2="86.36" y2="113.03" width="0.1524" layer="91"/>
-<junction x="86.36" y="116.84"/>
-<label x="99.06" y="116.84" size="1.778" layer="95"/>
-<pinref part="P+1" gate="1" pin="VCC"/>
-<pinref part="U1" gate="G$1" pin="3V3OUT"/>
-<pinref part="C1" gate="G$1" pin="1"/>
-</segment>
-<segment>
-<wire x1="185.42" y1="114.3" x2="185.42" y2="116.84" width="0.1524" layer="91"/>
-<wire x1="185.42" y1="116.84" x2="177.8" y2="116.84" width="0.1524" layer="91"/>
-<label x="177.8" y="116.84" size="1.778" layer="95"/>
-<pinref part="SJ2" gate="G$1" pin="3"/>
-</segment>
-</net>
 <net name="TXLED" class="0">
 <segment>
@@
 </segment>
 <segment>
-<pinref part="SJ2" gate="G$1" pin="2"/>
-<wire x1="190.5" y1="109.22" x2="203.2" y2="109.22" width="0.1524" layer="91"/>
+<wire x1="198.12" y1="109.22" x2="210.82" y2="109.22" width="0.1524" layer="91"/>
 <label x="195.58" y="111.76" size="1.778" layer="95"/>
 <pinref part="J1" gate="G$1" pin="4"/>
-<wire x1="203.2" y1="109.22" x2="205.74" y2="109.22" width="0.1524" layer="91"/>
+<wire x1="210.82" y1="109.22" x2="205.74" y2="109.22" width="0.1524" layer="91"/>
 <wire x1="220.98" y1="109.22" x2="205.74" y2="109.22" width="0.1524" layer="91"/>
+<pinref part="S1" gate="1" pin="P"/>
+<wire x1="193.04" y1="109.22" x2="220.98" y2="109.22" width="0.1524" layer="91"/>
+<junction x="220.98" y="109.22"/>
 </segment>
 </net>
@@
 </segment>
 <segment>
-<wire x1="185.42" y1="104.14" x2="185.42" y2="101.6" width="0.1524" layer="91"/>
-<wire x1="185.42" y1="101.6" x2="177.8" y2="101.6" width="0.1524" layer="91"/>
-<label x="177.8" y="101.6" size="1.778" layer="95"/>
-<pinref part="SJ2" gate="G$1" pin="1"/>
+<pinref part="S1" gate="1" pin="O"/>
+<wire x1="185.42" y1="106.68" x2="185.42" y2="99.06" width="0.1524" layer="91"/>
+<label x="185.42" y="101.6" size="1.778" layer="95"/>
 </segment>
 </net>
@@
 </schematic>
 </drawing>
+<compatibility>
+<note version="8.2" severity="warning">
+Since Version 8.2, EAGLE supports online libraries. The ids
+of those online libraries will not be understood (or retained)
+with this version.
+</note>
+<note version="8.3" severity="warning">
+Since Version 8.3, EAGLE supports URNs for individual library
+assets (packages, symbols, and devices). The URNs of those assets
+will not be understood (or retained) with this version.
+</note>
+<note version="8.3" severity="warning">
+Since Version 8.3, EAGLE supports the association of 3D packages
+with devices in libraries, schematics, and board files. Those 3D
+packages will not be understood (or retained) with this version.
+</note>
+</compatibility>
 </eagle>

Commit message: Fixes to power.
Connections:
- new net N$4: U1.VCC, U1.VCCIO
- net 5V: no longer U1.VCC
- net POWER: no longer U1.VCCIO
Changed lines of the file:
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@@
 <?xml version="1.0" encoding="utf-8"?>
 <!DOCTYPE eagle SYSTEM "eagle.dtd">
-<eagle version="9.1.0">
+<eagle version="9.0.0">
 <drawing>
 <settings>
@@
 <net name="POWER" class="0">
 <segment>
-<wire x1="101.6" y1="114.3" x2="109.22" y2="114.3" width="0.1524" layer="91"/>
-<pinref part="U1" gate="G$1" pin="VCCIO"/>
-<label x="101.6" y="114.3" size="1.27" layer="95" rot="R180" xref="yes"/>
-</segment>
-<segment>
-<wire x1="198.12" y1="109.22" x2="210.82" y2="109.22" width="0.1524" layer="91"/>
-<label x="195.58" y="111.76" size="1.778" layer="95"/>
+<wire x1="198.12" y1="109.22" x2="205.74" y2="109.22" width="0.1524" layer="91"/>
+<label x="193.04" y="111.76" size="1.778" layer="95"/>
 <pinref part="J1" gate="G$1" pin="4"/>
 <wire x1="210.82" y1="109.22" x2="205.74" y2="109.22" width="0.1524" layer="91"/>
-<wire x1="220.98" y1="109.22" x2="205.74" y2="109.22" width="0.1524" layer="91"/>
+<wire x1="220.98" y1="109.22" x2="210.82" y2="109.22" width="0.1524" layer="91"/>
 <pinref part="S1" gate="1" pin="P"/>
 <wire x1="193.04" y1="109.22" x2="220.98" y2="109.22" width="0.1524" layer="91"/>
@@
 <wire x1="76.2" y1="129.54" x2="93.98" y2="129.54" width="0.1524" layer="91"/>
 <wire x1="93.98" y1="129.54" x2="93.98" y2="119.38" width="0.1524" layer="91"/>
-<wire x1="93.98" y1="119.38" x2="109.22" y2="119.38" width="0.1524" layer="91"/>
 <wire x1="76.2" y1="115.57" x2="76.2" y2="129.54" width="0.1524" layer="91"/>
 <wire x1="66.04" y1="113.03" x2="66.04" y2="129.54" width="0.1524" layer="91"/>
@@
 <junction x="76.2" y="129.54"/>
 <junction x="93.98" y="129.54"/>
-<label x="99.06" y="119.38" size="1.778" layer="95"/>
-<pinref part="U1" gate="G$1" pin="VCC"/>
 <pinref part="C5" gate="G$1" pin="+"/>
 <pinref part="C2" gate="G$1" pin="1"/>
@@
 </segment>
 </net>
+<net name="N$4" class="0">
+<segment>
+<wire x1="93.98" y1="119.38" x2="93.98" y2="121.92" width="0.1524" layer="91"/>
+<pinref part="U1" gate="G$1" pin="VCC"/>
+<wire x1="109.22" y1="119.38" x2="93.98" y2="119.38" width="0.1524" layer="91"/>
+<junction x="93.98" y="119.38"/>
+<pinref part="U1" gate="G$1" pin="VCCIO"/>
+<wire x1="109.22" y1="114.3" x2="93.98" y2="114.3" width="0.1524" layer="91"/>
+<wire x1="93.98" y1="114.3" x2="93.98" y2="119.38" width="0.1524" layer="91"/>
+</segment>
+</net>

Commit message: Upgrade to 9.1.1 and fixes
Connections:
- net POWER renamed N$5
Changed lines of the file:
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@@
 <?xml version="1.0" encoding="utf-8"?>
 <!DOCTYPE eagle SYSTEM "eagle.dtd">
-<eagle version="9.0.0">
+<eagle version="9.1.1">
 <drawing>
 <settings>
@@
 </segment>
 </net>
-<net name="POWER" class="0">
-<segment>
-<wire x1="198.12" y1="109.22" x2="205.74" y2="109.22" width="0.1524" layer="91"/>
-<label x="193.04" y="111.76" size="1.778" layer="95"/>
-<pinref part="J1" gate="G$1" pin="4"/>
-<wire x1="210.82" y1="109.22" x2="205.74" y2="109.22" width="0.1524" layer="91"/>
-<wire x1="220.98" y1="109.22" x2="210.82" y2="109.22" width="0.1524" layer="91"/>
-<pinref part="S1" gate="1" pin="P"/>
-<wire x1="193.04" y1="109.22" x2="220.98" y2="109.22" width="0.1524" layer="91"/>
-<junction x="220.98" y="109.22"/>
-</segment>
-</net>
 <net name="5V" class="0">
 <segment>
@@
 </segment>
 </net>
+<net name="N$5" class="0">
+<segment>
+<pinref part="S1" gate="1" pin="P"/>
+<pinref part="J1" gate="G$1" pin="4"/>
+<wire x1="193.04" y1="109.22" x2="220.98" y2="109.22" width="0.1524" layer="91"/>
+</segment>
+</net>

Commit message: new FTDI FT232RL for manufacturing
Parts:
- renumbered C5 to C1
Connections:
- net N$5 renamed 5V-J1
- removed net N$4: U1.VCC, U1.VCCIO
- net 5V: now also U1.VCC, U1.VCCIO
Changed lines of the file:
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@@
 <?xml version="1.0" encoding="utf-8"?>
 <!DOCTYPE eagle SYSTEM "eagle.dtd">
-<eagle version="9.1.1">
+<eagle version="9.1.0">
 <drawing>
 <settings>
@@
 <parts>
 <part name="C2" library="openSX70_PATHFINDER_V5.5-SEEED_20180522" deviceset="CERAMIC-100NF-50V-10%-X7R(0603)" device="" value="100nf"/>
-<part name="C5" library="Seeed-Capacitor-2016" deviceset="TANTALUM-SMD-10UF-16V-10%(AVX-A)" device="" value="10uf"/>
+<part name="C1" library="Seeed-Capacitor-2016" deviceset="TANTALUM-SMD-10UF-16V-10%(AVX-A)" device="" value="10uf"/>
 <part name="GND2" library="SparkFun" deviceset="GND" device=""/>
 <part name="FRAME1" library="SparkFun-Aesthetics" deviceset="FRAME-LETTER" device=""/>
@@
 <instances>
 <instance part="C2" gate="G$1" x="66.04" y="109.22" rot="R270"/>
-<instance part="C5" gate="G$1" x="76.2" y="111.76" rot="R270"/>
+<instance part="C1" gate="G$1" x="76.2" y="111.76" rot="R270"/>
 <instance part="GND2" gate="1" x="106.68" y="86.36"/>
 <instance part="FRAME1" gate="G$1" x="0" y="0"/>
@@
 <segment>
 <wire x1="76.2" y1="104.14" x2="76.2" y2="107.95" width="0.1524" layer="91"/>
-<pinref part="C5" gate="G$1" pin="-"/>
+<pinref part="C1" gate="G$1" pin="-"/>
 <pinref part="GND8" gate="1" pin="GND"/>
 </segment>
@@
 <junction x="76.2" y="129.54"/>
 <junction x="93.98" y="129.54"/>
-<pinref part="C5" gate="G$1" pin="+"/>
+<pinref part="C1" gate="G$1" pin="+"/>
 <pinref part="C2" gate="G$1" pin="1"/>
 <pinref part="U$3" gate="G$1" pin="5V"/>
@@
 <label x="185.42" y="101.6" size="1.778" layer="95"/>
 </segment>
-</net>
-<net name="N$3" class="0">
-<segment>
-<pinref part="U1" gate="G$1" pin="USBDM"/>
-<wire x1="109.22" y1="127" x2="53.34" y2="127" width="0.1524" layer="91"/>
-<pinref part="USB1" gate="G$1" pin="DM"/>
-<wire x1="53.34" y1="127" x2="53.34" y2="124.46" width="0.1524" layer="91"/>
-<wire x1="53.34" y1="124.46" x2="41.91" y2="124.46" width="0.1524" layer="91"/>
-</segment>
-</net>
-<net name="N$4" class="0">
 <segment>
 <wire x1="93.98" y1="119.38" x2="93.98" y2="121.92" width="0.1524" layer="91"/>
@@
 <wire x1="109.22" y1="114.3" x2="93.98" y2="114.3" width="0.1524" layer="91"/>
 <wire x1="93.98" y1="114.3" x2="93.98" y2="119.38" width="0.1524" layer="91"/>
-</segment>
-</net>
-<net name="N$5" class="0">
+<label x="101.6" y="116.84" size="1.778" layer="95"/>
+<label x="101.6" y="111.76" size="1.778" layer="95"/>
+</segment>
+</net>
+<net name="N$3" class="0">
+<segment>
+<pinref part="U1" gate="G$1" pin="USBDM"/>
+<wire x1="109.22" y1="127" x2="53.34" y2="127" width="0.1524" layer="91"/>
+<pinref part="USB1" gate="G$1" pin="DM"/>
+<wire x1="53.34" y1="127" x2="53.34" y2="124.46" width="0.1524" layer="91"/>
+<wire x1="53.34" y1="124.46" x2="41.91" y2="124.46" width="0.1524" layer="91"/>
+</segment>
+</net>
+<net name="5V-J1" class="0">
 <segment>
 <pinref part="S1" gate="1" pin="P"/>
 <pinref part="J1" gate="G$1" pin="4"/>
 <wire x1="193.04" y1="109.22" x2="220.98" y2="109.22" width="0.1524" layer="91"/>
-</segment>
-</net>
+<label x="198.12" y="111.76" size="1.778" layer="95"/>
+</segment>
+</net>
