File: FT231X/ft231x-breakout-v11-openSX70versionSEEED.sch (EAGLE design)
At the start: 24 parts, among them J1 XF2L-0625-1, Q1 2N7002, U1 FTS31XS-U

Commit message: NEW FTDI for manufacture 232RL based on Sparkfun FTDI basic
Parts:
- removed SJ1, SJ4: (no value), SparkFun-Passives:SOLDERJUMPER_2WAYS
- removed SJ2: TXLED, SparkFun-Passives:SOLDERJUMPERTRACE
- removed SJ3: RXLED, SparkFun-Passives:JUMPER-PAD-2-NC_BY_TRACE
Connections:
- removed net N$10: J1-3.MS, SJ4.2
- removed net N$7: R3.1, SJ2.2
- removed net N$8: R4.1, SJ3.2
- net 3.3V: no longer SJ1.1
- net RXLED: now also R4.1; no longer SJ3.1
- net TXLED: now also R3.1; no longer SJ2.1
- net VCC: no longer SJ1.3
- net VOUT: now also J1-3.MS; no longer SJ1.2, SJ4.3
Other:
- note removed: "CUT TRACE ON SJ1 TO SWITCH VOUT FROM 5V TO 3.3V"
- note removed: "DO NOT CONNECT ALL THREE PADS ON SJ1 AT THE SAME TIME!"
Changed lines of the file:
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@@
 <?xml version="1.0" encoding="utf-8"?>
 <!DOCTYPE eagle SYSTEM "eagle.dtd">
-<eagle version="9.0.0">
+<eagle version="9.1.0">
 <drawing>
 <settings>
@@
 <part name="GND7" library="SparkFun-Aesthetics" deviceset="GND" device=""/>
 <part name="GND8" library="SparkFun-Aesthetics" deviceset="GND" device=""/>
-<part name="SJ1" library="SparkFun-Passives" deviceset="SOLDERJUMPER_2WAY" device="S"/>
 <part name="P+5" library="SparkFun-Aesthetics" deviceset="3.3V" device=""/>
-<part name="P+6" library="SparkFun-Aesthetics" deviceset="VCC" device=""/>
-<part name="P+7" library="SparkFun-Aesthetics" deviceset="3.3V" device=""/>
 <part name="P+1" library="SparkFun-Aesthetics" deviceset="VCC" device=""/>
 <part name="C1" library="Seeed-Capacitor-2016" deviceset="TANTALUM-SMD-10UF-16V-10%(AVX-B)" device="" value="10uf"/>
@@
 <part name="P+8" library="SparkFun-Aesthetics" deviceset="3.3V" device=""/>
 <part name="P+9" library="SparkFun-Aesthetics" deviceset="3.3V" device=""/>
-<part name="SJ2" library="SparkFun-Passives" deviceset="SOLDERJUMPER" device="TRACE" value="TXLED"/>
-<part name="SJ3" library="SparkFun-Passives" deviceset="JUMPER-PAD-2-NC_BY_TRACE" device="" value="RXLED"/>
 <part name="Q1" library="Seeed-Transistor" deviceset="SMD-MOSFET-N-CH-60V-300MA-LOGIC-LEVEL-FET-2N7002(SOT-23)" device="" value="2N7002"/>
 <part name="R5" library="Seeed-Resistor" deviceset="SMD-RES-10K-5%-1/10W(0603)" device="" value="10K 1/10W"/>
@@
 <part name="JP5" library="SparkFun-Aesthetics" deviceset="FIDUCIAL" device="1X2" value="FIDUCIAL1X2"/>
 <part name="J1" library="con-omron" library_urn="urn:adsk.eagle:library:167" deviceset="XF2*-06?" device="25-1" package3d_urn="urn:adsk.eagle:package:9011/1" technology="L"/>
-<part name="SJ4" library="SparkFun-Passives" deviceset="SOLDERJUMPER_2WAY" device="S"/>
 <part name="D3" library="Seeed-LED" deviceset="SMD-LED-CLEAR-YELLOW(0603)" device="" value="YELLOW-0603"/>
 <part name="D2" library="Seeed-LED" deviceset="LED-SMD-RED-DIFFUSED(0603)" device="" value="RED-0603"/>
+<part name="P+11" library="SparkFun-Aesthetics" deviceset="VCC" device=""/>
 </parts>
 <sheets>
 <sheet>
 <plain>
-<wire x1="220.98" y1="160.02" x2="220.98" y2="161.798" width="1.016" layer="94"/>
-<wire x1="114.3" y1="128.778" x2="114.3" y2="130.302" width="1.016" layer="94"/>
-<wire x1="106.68" y1="128.778" x2="106.68" y2="130.302" width="1.016" layer="94"/>
 <wire x1="0" y1="93.98" x2="134.62" y2="93.98" width="0.127" layer="97" style="shortdash"/>
 <wire x1="134.62" y1="93.98" x2="134.62" y2="185.42" width="0.127" layer="97" style="shortdash"/>
@@
 <text x="93.98" y="167.64" size="1.778" layer="97">CUT TRACES ON SJ2 AND SJ3
      TO DISCONNECT LEDS</text>
-<text x="198.12" y="175.26" size="1.778" layer="97">CUT TRACE ON SJ1 TO SWITCH
-      VOUT FROM 5V TO 3.3V</text>
-<text x="195.58" y="142.24" size="1.778" layer="97">DO NOT CONNECT ALL THREE PADS
-      ON SJ1 AT THE SAME TIME!</text>
 </plain>
 <instances>
@@
 <instance part="GND7" gate="1" x="220.98" y="109.22"/>
 <instance part="GND8" gate="1" x="96.52" y="81.28" rot="R180"/>
-<instance part="SJ1" gate="G$1" x="220.98" y="160.02" rot="R180"/>
 <instance part="P+5" gate="G$1" x="53.34" y="152.4" smashed="yes">
 <attribute name="VALUE" x="51.054" y="155.194" size="1.778" layer="96"/>
-</instance>
-<instance part="P+6" gate="G$1" x="220.98" y="167.64" smashed="yes">
-<attribute name="VALUE" x="219.456" y="170.688" size="1.778" layer="96"/>
-</instance>
-<instance part="P+7" gate="G$1" x="210.82" y="167.64" smashed="yes">
-<attribute name="VALUE" x="208.534" y="170.688" size="1.778" layer="96"/>
 </instance>
 <instance part="P+1" gate="G$1" x="30.48" y="157.48"/>
@@
 <instance part="P+9" gate="G$1" x="106.68" y="160.02" smashed="yes">
 <attribute name="VALUE" x="104.394" y="162.814" size="1.778" layer="96"/>
-</instance>
-<instance part="SJ2" gate="1" x="121.92" y="124.46" smashed="yes" rot="R90">
-<attribute name="NAME" x="119.38" y="121.92" size="1.778" layer="95" rot="R90"/>
-</instance>
-<instance part="SJ3" gate="G$1" x="106.68" y="129.54" smashed="yes" rot="R90">
-<attribute name="NAME" x="104.14" y="127" size="1.778" layer="95" rot="R90"/>
 </instance>
 <instance part="Q1" gate="G$1" x="160.02" y="134.62" rot="R270"/>
@@
 <instance part="J1" gate="-5" x="101.6" y="68.58"/>
 <instance part="J1" gate="-6" x="101.6" y="66.04"/>
-<instance part="SJ4" gate="G$1" x="66.04" y="71.12" rot="R180"/>
 <instance part="D3" gate="G$1" x="121.92" y="154.94" rot="R270"/>
 <instance part="D2" gate="G$1" x="106.68" y="152.4" rot="R270"/>
+<instance part="P+11" gate="G$1" x="205.74" y="160.02" smashed="yes" rot="R90">
+<attribute name="VALUE" x="202.692" y="158.496" size="1.778" layer="96" rot="R90"/>
+</instance>
 </instances>
 <busses>
@@
 <pinref part="P+3" gate="G$1" pin="VCC"/>
 <wire x1="210.82" y1="124.46" x2="210.82" y2="120.65" width="0.1524" layer="91"/>
-</segment>
-<segment>
-<pinref part="SJ1" gate="G$1" pin="3"/>
-<pinref part="P+6" gate="G$1" pin="VCC"/>
-<wire x1="220.98" y1="167.64" x2="220.98" y2="165.1" width="0.1524" layer="91"/>
 </segment>
 <segment>
@@
 </segment>
 <segment>
-<pinref part="SJ1" gate="G$1" pin="1"/>
-<wire x1="220.98" y1="154.94" x2="220.98" y2="152.4" width="0.1524" layer="91"/>
-<pinref part="P+7" gate="G$1" pin="3.3V"/>
-<wire x1="220.98" y1="152.4" x2="210.82" y2="152.4" width="0.1524" layer="91"/>
-<wire x1="210.82" y1="152.4" x2="210.82" y2="167.64" width="0.1524" layer="91"/>
-</segment>
-<segment>
 <pinref part="P+8" gate="G$1" pin="3.3V"/>
 <pinref part="D3" gate="G$1" pin="+"/>
@@
 <wire x1="86.36" y1="119.38" x2="121.92" y2="119.38" width="0.1524" layer="91"/>
 <label x="98.298" y="119.634" size="1.778" layer="95"/>
-<pinref part="SJ2" gate="1" pin="1"/>
+<pinref part="R3" gate="G$1" pin="1"/>
+<wire x1="121.92" y1="133.35" x2="121.92" y2="129.54" width="0.1524" layer="91"/>
+<wire x1="121.92" y1="129.54" x2="121.92" y2="119.38" width="0.1524" layer="91"/>
 </segment>
 </net>
@@
 <wire x1="86.36" y1="121.92" x2="106.68" y2="121.92" width="0.1524" layer="91"/>
 <label x="98.044" y="122.174" size="1.778" layer="95"/>
-<pinref part="SJ3" gate="G$1" pin="1"/>
 <wire x1="106.68" y1="121.92" x2="106.68" y2="124.46" width="0.1524" layer="91"/>
+<pinref part="R4" gate="G$1" pin="1"/>
+<wire x1="106.68" y1="134.62" x2="106.68" y2="138.43" width="0.1524" layer="91"/>
+<wire x1="106.68" y1="134.62" x2="106.68" y2="124.46" width="0.1524" layer="91"/>
 </segment>
 </net>
@@
 <wire x1="106.68" y1="148.59" x2="106.68" y2="146.05" width="0.1524" layer="91"/>
 <junction x="106.68" y="148.59"/>
-</segment>
-</net>
-<net name="N$7" class="0">
-<segment>
-<pinref part="R3" gate="G$1" pin="1"/>
-<pinref part="SJ2" gate="1" pin="2"/>
-<wire x1="121.92" y1="133.35" x2="121.92" y2="129.54" width="0.1524" layer="91"/>
-</segment>
-</net>
-<net name="N$8" class="0">
-<segment>
-<pinref part="R4" gate="G$1" pin="1"/>
-<pinref part="SJ3" gate="G$1" pin="2"/>
-<wire x1="106.68" y1="134.62" x2="106.68" y2="138.43" width="0.1524" layer="91"/>
 </segment>
 </net>
@@
 <net name="VOUT" class="0">
 <segment>
-<pinref part="SJ1" gate="G$1" pin="2"/>
-<wire x1="226.06" y1="160.02" x2="228.6" y2="160.02" width="0.1524" layer="91"/>
-<label x="228.6" y="160.02" size="1.27" layer="95" xref="yes"/>
-</segment>
-<segment>
 <pinref part="R6" gate="G$1" pin="2"/>
 <wire x1="167.64" y1="152.4" x2="167.64" y2="146.05" width="0.1524" layer="91"/>
@@
 </segment>
 <segment>
-<label x="48.26" y="78.74" size="1.778" layer="95"/>
-<pinref part="SJ4" gate="G$1" pin="3"/>
-<wire x1="66.04" y1="76.2" x2="48.26" y2="76.2" width="0.1524" layer="91"/>
-</segment>
-</net>
-<net name="N$10" class="0">
+<pinref part="P+11" gate="G$1" pin="VCC"/>
+<wire x1="205.74" y1="160.02" x2="226.06" y2="160.02" width="0.1524" layer="91"/>
+<label x="226.06" y="165.1" size="1.778" layer="95"/>
+</segment>
 <segment>
 <pinref part="J1" gate="-3" pin="MS"/>
 <wire x1="71.12" y1="73.66" x2="99.06" y2="73.66" width="0.1524" layer="91"/>
-<pinref part="SJ4" gate="G$1" pin="2"/>
-<wire x1="71.12" y1="73.66" x2="71.12" y2="71.12" width="0.1524" layer="91"/>
-</segment>
-</net>
+<label x="73.66" y="76.2" size="1.778" layer="95"/>
+</segment>
+</net>
